Commit message: Placed Cyton on top

File: be_description/urdf/be.urdf (robot description, URDF)
Before this commit: robot be, 10 links, 9 joints
Links:
- added link cyton_base_link, mass 9; collision mesh filename=package://cyton_gamma_300_description/meshes/gamma_base.dae; visual mesh filename=package://cyton_gamma_300_description/meshes/gamma_base.dae
- added link elbow_pitch, mass 1; collision mesh filename=package://cyton_gamma_300_description/meshes/Elbow_Pitch.dae; visual mesh filename=package://cyton_gamma_300_description/meshes/Elbow_Pitch.dae
- added link elbow_roll, mass 1; collision mesh filename=package://cyton_gamma_300_description/meshes/Elbow_Roll.dae; visual mesh filename=package://cyton_gamma_300_description/meshes/Elbow_Roll.dae
- added link elbow_yaw, mass 1; collision mesh filename=package://cyton_gamma_300_description/meshes/Elbow_Yaw.dae; visual mesh filename=package://cyton_gamma_300_description/meshes/Elbow_Yaw.dae
- added link gripper_finger1, mass 0.5; collision mesh filename=package://cyton_gamma_300_description/meshes/Gripper_Finger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; visual mesh filename=package://cyton_gamma_300_description/meshes/Gripper_Finger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
- added link gripper_finger2, mass 0.5; collision mesh filename=package://cyton_gamma_300_description/meshes/Gripper_Finger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; visual mesh filename=package://cyton_gamma_300_description/meshes/Gripper_Finger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
- added link shoulder_pitch, mass 1; collision mesh filename=package://cyton_gamma_300_description/meshes/Shoulder_Pitch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; visual mesh filename=package://cyton_gamma_300_description/meshes/Shoulder_Pitch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
- added link shoulder_roll, mass 1; collision mesh filename=package://cyton_gamma_300_description/meshes/Shoulder_Roll.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; visual mesh filename=package://cyton_gamma_300_description/meshes/Shoulder_Roll.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
- added link virtual_endeffector, mass 0.03; visual sphere radius=0.01
- added link wrist_pitch, mass 1; collision mesh filename=package://cyton_gamma_300_description/meshes/Wrist_Pitch.dae; visual mesh filename=package://cyton_gamma_300_description/meshes/Wrist_Pitch.dae
- added link wrist_roll, mass 1; collision mesh filename=package://cyton_gamma_300_description/meshes/Wrist_Roll.dae; visual mesh filename=package://cyton_gamma_300_description/meshes/Wrist_Roll.dae
Joints:
- added joint cyton_gamma_300: type fixed, parent base_link, child cyton_base_link, origin xyz=0.08 0 0.24 rpy=0 0 0
- added joint elbow_pitch_joint: type revolute, parent elbow_roll, child elbow_pitch, origin xyz=0 0 0.052 rpy=1.2 0 0, axis 1 0 0, limit lower=-3.2 upper=0.8 effort=100.0 velocity=1.0
- added joint elbow_roll_joint: type revolute, parent shoulder_pitch, child elbow_roll, origin xyz=0 0 0.089 rpy=0 0 1.2, axis 0 0 1, limit lower=-3.8 upper=1.4 effort=100.0 velocity=1.0
- added joint elbow_yaw_joint: type revolute, parent elbow_pitch, child elbow_yaw, origin xyz=0 0 0.072 rpy=0 -1.2 0, axis 0 -1 0, limit lower=-3.2 upper=0.8 effort=100.0 velocity=1.0
- added joint gripper_finger1_joint: type prismatic, parent wrist_roll, child gripper_finger1, origin xyz=-0.01331 0.00485 0.077225 rpy=0 0 0, axis 1 0 0, limit lower=-0.008 upper=0.008 effort=100.0 velocity=1.0
- added joint gripper_finger2_joint: type prismatic, parent wrist_roll, child gripper_finger2, origin xyz=0.0098 0.00485 0.077225 rpy=0 0 0, axis 1 0 0, limit lower=-0.008 upper=0.008 effort=100.0 velocity=1.0, mimic joint=gripper_finger1_joint multiplier=-1
- added joint shoulder_pitch_joint: type revolute, parent shoulder_roll, child shoulder_pitch, origin xyz=0 0 0.063 rpy=1.2 0 0, axis 1 0 0, limit lower=-2.6 upper=0.2 effort=100.0 velocity=1.0
- added joint shoulder_roll_joint: type revolute, parent cyton_base_link, child shoulder_roll, origin xyz=0 0 0.05315 rpy=0 0 1.2, axis 0 0 1, limit lower=-3.9 upper=1.5 effort=100.0 velocity=1.0
- added joint virtual_endeffector_joint: type fixed, parent wrist_roll, child virtual_endeffector, origin xyz=-0.002316 0.0079 0.079425 rpy=0 0 0
- added joint wrist_pitch_joint: type revolute, parent elbow_yaw, child wrist_pitch, origin xyz=0 0 0.0718 rpy=1.2 0 0, axis 1 0 0, limit lower=-3.1 upper=0.8 effort=100.0 velocity=1.0
- added joint wrist_roll_joint: type revolute, parent wrist_pitch, child wrist_roll, origin xyz=0 0 0.051425 rpy=0 0 1.2, axis 0 0 1, limit lower=-3.8 upper=1.4 effort=100.0 velocity=1.0

File: be_description/urdf/be.xacro (robot description, xacro)
@@ -22,5 +22,8 @@
 	<!-- import the pioneer 3dx's wheels -->
 	<xacro:include filename="$(find p3dx_description)/urdf/pioneer3dx_wheel.xacro" />
+	<!-- import the materials -->
 	<xacro:include filename="$(find be_description)/urdf/materials.xacro" />
+	<!-- import cyton_gamma_300-->
+	<xacro:include filename="$(find be_description)/urdf/cyton_gamma_300.urdf.xacro" />
 	<!-- chassis -->
 	<link name="base_link">
@@ -191,3 +194,9 @@
 		<child link="front_sonar" />
 	</joint>
+	<!-- Connect arm to base -->
+  <joint name="cyton_gamma_300" type="fixed">
+    <parent link="base_link" />
+    <child link="cyton_base_link" />
+    <origin xyz="0.08 0 0.24" rpy="0 0 0" />
+  </joint>
 </robot>
